File: PCB/ESP32 Devoard.kicad_pcb (KiCad board)
At the start: 2 copper layers, 27.9 x 38.7 mm, 23 parts, among them J1 USB_C_Receptacle_USB2.0_16P, J2 Conn_01x20_Pin, J3 Conn_01x20_Pin, SW1 SW_Push, SW2 SW_Push, U2 AP63203WU, U3 ESP32-S3-WROOM-1

Commit message: Add files via upload
Parts:
- R3, R4: value 50 K -> 5.1 K
Connections:
- J1 pad SH: GND -> (no net)
Routing:
- net BOOT: track 11.2 -> 10.8 mm, vias 0 -> 1
- net +5V: track 38.8 -> 39.0 mm, vias 0 -> 3
- net +3.3V: vias 4 -> 5
Changed lines of the file:
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@@
 			(layers "*.Cu" "*.Mask")
 			(remove_unused_layers no)
-			(net "GND")
 		)
 		(pad "SH" thru_hole oval
@@
 			(layers "*.Cu" "*.Mask")
 			(remove_unused_layers no)
-			(net "GND")
 		)
 		(pad "SH" thru_hole oval
@@
 			(layers "*.Cu" "*.Mask")
 			(remove_unused_layers no)
-			(net "GND")
 		)
 		(pad "SH" thru_hole oval
@@
 			(layers "*.Cu" "*.Mask")
 			(remove_unused_layers no)
-			(net "GND")
 		)
 		(embedded_fonts no)
@@
 			)
 		)
-		(property "Value" "50 K"
+		(property "Value" "5.1 K"
 			(at 0 1.43 90)
 			(layer "F.Fab")
@@
 			)
 		)
-		(property "Value" "50 K"
+		(property "Value" "5.1 K"
 			(at 0 1.43 90)
 			(layer "F.Fab")
@@
 		(net "+3.3V")
 	)
-	(segment
-		(start 101.51 58.96)
-		(end 99.06 58.96)
-		(width 0.2)
-		(layer "F.Cu")
-		(net "+3.3V")
-	)
 	(via
 		(at 117.45 85.445)
@@
 	)
 	(via
+		(at 101.51 58.96)
+		(size 0.6)
+		(drill 0.3)
+		(layers "F.Cu" "B.Cu")
+		(net "+3.3V")
+	)
+	(via
 		(at 104.53 68.59)
 		(size 0.6)
@@
 	)
 	(segment
+		(start 99.06 58.96)
+		(end 101.51 58.96)
+		(width 0.2)
+		(layer "B.Cu")
+		(net "+3.3V")
+	)
+	(segment
 		(start 99.06 69.96)
 		(end 103.16 69.96)
@@
 	)
 	(segment
-		(start 123.76 70.96)
-		(end 124.46 70.96)
+		(start 122.39 73.24)
+		(end 122.39 72.541472)
 		(width 0.2)
 		(layer "F.Cu")
@@
 	)
 	(segment
-		(start 120.51 78.76)
-		(end 119.92 79.35)
+		(start 120.88 74.75)
+		(end 122.39 73.24)
 		(width 0.2)
 		(layer "F.Cu")
@@
 	)
 	(segment
-		(start 122.19 72.53)
-		(end 123.76 70.96)
+		(start 120.51 78.76)
+		(end 119.92 79.35)
 		(width 0.2)
 		(layer "F.Cu")
@@
 	(segment
 		(start 120.51 74.75)
-		(end 121.46 74.75)
+		(end 120.88 74.75)
 		(width 0.2)
 		(layer "F.Cu")
@@
 	)
 	(segment
-		(start 122.19 74.02)
-		(end 122.19 72.53)
+		(start 120.51 74.75)
+		(end 120.51 78.76)
 		(width 0.2)
 		(layer "F.Cu")
 		(net "BOOT")
 	)
+	(via
+		(at 122.39 72.541472)
+		(size 0.6)
+		(drill 0.3)
+		(layers "F.Cu" "B.Cu")
+		(net "BOOT")
+	)
 	(segment
-		(start 120.51 74.75)
-		(end 120.51 78.76)
+		(start 122.39 72.541472)
+		(end 123.971472 70.96)
 		(width 0.2)
-		(layer "F.Cu")
+		(layer "B.Cu")
 		(net "BOOT")
 	)
 	(segment
-		(start 121.46 74.75)
-		(end 122.19 74.02)
+		(start 123.971472 70.96)
+		(end 124.46 70.96)
 		(width 0.2)
-		(layer "F.Cu")
+		(layer "B.Cu")
 		(net "BOOT")
 	)
@@
 	)
 	(segment
-		(start 108.4 92.16)
-		(end 109.765 90.795)
+		(start 110 89.48)
+		(end 110 88.06)
 		(width 0.3)
 		(layer "F.Cu")
@@
 	)
 	(segment
-		(start 110 88.135832)
-		(end 112.320832 85.815)
+		(start 108.4 92.16)
+		(end 109.765 90.795)
 		(width 0.3)
 		(layer "F.Cu")
@@
 	)
 	(segment
+		(start 111.08 86.665)
+		(end 111.08 86.97)
+		(width 0.3)
+		(layer "F.Cu")
+		(net "+5V")
+	)
+	(segment
 		(start 113.8 85.445)
 		(end 113.43 85.815)
@@
 	)
 	(segment
+		(start 112.303694 85.742448)
+		(end 112.002552 85.742448)
+		(width 0.3)
+		(layer "F.Cu")
+		(net "+5V")
+	)
+	(segment
 		(start 98.963984 70.96)
 		(end 98.285 71.638984)
@@
 	)
 	(segment
+		(start 110 88.06)
+		(end 110.09 87.97)
+		(width 0.3)
+		(layer "F.Cu")
+		(net "+5V")
+	)
+	(segment
+		(start 112.002552 85.742448)
+		(end 111.08 86.665)
+		(width 0.3)
+		(layer "F.Cu")
+		(net "+5V")
+	)
+	(segment
 		(start 98.285 71.638984)
 		(end 98.285 82.594999)
@@
 		(net "+5V")
 	)
+	(via
+		(at 110.09 87.97)
+		(size 0.6)
+		(drill 0.3)
+		(layers "F.Cu" "B.Cu")
+		(net "+5V")
+	)
+	(via
+		(at 111.08 86.97)
+		(size 0.6)
+		(drill 0.3)
+		(layers "F.Cu" "B.Cu")
+		(net "+5V")
+	)
+	(via
+		(at 112.303694 85.742448)
+		(size 0.6)
+		(drill 0.3)
+		(layers "F.Cu" "B.Cu")
+		(net "+5V")
+	)
 	(segment
-		(start 110 89.48)
-		(end 110 88.135832)
+		(start 110.09 87.97)
+		(end 110.09 87.96)
 		(width 0.3)
-		(layer "F.Cu")
+		(layer "B.Cu")
+		(net "+5V")
+	)
+	(segment
+		(start 110.09 87.96)
+		(end 111.08 86.97)
+		(width 0.3)
+		(layer "B.Cu")
 		(net "+5V")
 	)
@@
 	)
 	(segment
+		(start 104.28 60.78)
+		(end 103.01 60.78)
+		(width 0.2)
+		(layer "F.Cu")
+		(net "EN")
+	)
+	(segment
 		(start 101.33 59.96)
 		(end 99.06 59.96)
@@
 	)
 	(segment
-		(start 107.29 63.54)
-		(end 104.53 60.78)
+		(start 104.47 60.97)
+		(end 104.28 60.78)
 		(width 0.2)
 		(layer "F.Cu")
@@
 	)
 	(segment
-		(start 107.29 68.7)
-		(end 107.29 63.54)
-		(width 0.2)
-		(layer "F.Cu")
-		(net "EN")
-	)
-	(segment
-		(start 104.53 60.78)
-		(end 103.01 60.78)
-		(width 0.2)
-		(layer "F.Cu")
-		(net "EN")
-	)
-	(segment
 		(start 100.56 79.325)
 		(end 102.415 79.325)
@@
 	)
 	(segment
-		(start 110.5 71.91)
-		(end 107.29 68.7)
-		(width 0.2)
-		(layer "F.Cu")
-		(net "EN")
-	)
-	(segment
 		(start 110.7 79.38)
 		(end 106.62 79.38)
@@
 	)
 	(via
-		(at 110.5 71.91)
+		(at 104.47 60.97)
 		(size 0.6)
 		(drill 0.3)
@@
 	)
 	(segment
-		(start 110.72 78.66)
-		(end 110.72 72.13)
+		(start 104.47 60.97)
+		(end 104.47 65.88)
 		(width 0.2)
 		(layer "B.Cu")
@@
 	)
 	(segment
-		(start 110.72 72.13)
-		(end 110.5 71.91)
+		(start 104.47 65.88)
+		(end 110.72 72.13)
 		(width 0.2)
 		(layer "B.Cu")
@@
 		(width 0.2)
 		(layer "B.Cu")
+		(net "EN")
+	)
+	(segment
+		(start 110.72 72.13)
+		(end 110.72 78.66)
+		(width 0.2)
+		(layer "B.Cu")

Commit message: Add files via upload
Parts:
- J2, J3: footprint Connector_PinHeader_1.00mm:PinHeader_1x20_P1.00mm_Vertical -> Connector_PinHeader_2.54mm:PinHeader_1x20_P2.54mm_Vertical
- moved J3 30.2 mm to (129.5, 106.7)
- moved R1 14.3 mm to (107.2, 100.3)
- moved R2 14.3 mm to (108.8, 100.3)
- moved R3 14.3 mm to (105.5, 100.3)
- moved R4 14.3 mm to (110.4, 100.3)
- moved J1 14.1 mm to (108.0, 107.3)
- moved J2 5.10 mm to (94.0, 58.4)
- moved C5 0.69 mm to (121.8, 85.5), turned to -90 degrees
- moved C4 0.65 mm to (121.0, 85.5), turned to -90 degrees
- moved L1 0.21 mm to (119.9, 84.3)
Connections:
- J1 pad SH: (no net) -> GND
Routing:
- net +5V: track 39.0 -> 68.8 mm, vias 3 -> 8
- net I011: track 10.8 -> 36.4 mm
- net I012: track 13.0 -> 38.2 mm, vias 1 -> 3
- net I013: track 14.7 -> 37.9 mm
- net I014: track 13.6 -> 34.7 mm
- net I021: track 12.5 -> 33.2 mm
- net I010: track 13.7 -> 33.5 mm, vias 1 -> 3
- net I09: track 12.6 -> 31.6 mm, vias 1 -> 3
- net I047: track 11.1 -> 30.1 mm
- net I048: track 9.42 -> 28.3 mm
- net I046: track 11.7 -> 28.5 mm, vias 1 -> 3
- net I045: track 7.39 -> 24.1 mm, vias 1 -> 3
- net _D-: track 16.6 -> 31.1 mm
- net _D+: track 15.8 -> 30.2 mm
- net I03: track 11.7 -> 25.5 mm, vias 1 -> 3
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Other:
- board size 27.9 x 38.7 mm -> 41.1 x 53.2 mm

Commit message: Add files via upload
Parts:
- C1, C2, C3, C4, C5: footprint Capacitor_SMD:C_0201_0603Metric -> Capacitor_SMD:C_0402_1005Metric
- C6, C7: footprint Capacitor_SMD:C_0805_2012Metric -> Capacitor_SMD:C_0402_1005Metric
- D1: footprint LED_SMD:LED_0201_0603Metric -> Capacitor_SMD:C_0402_1005Metric
- R5, R6: footprint Resistor_SMD:R_0805_2012Metric -> Capacitor_SMD:C_0402_1005Metric
- R7: footprint Resistor_SMD:R_0201_0603Metric_Pad0.64x0.40mm_HandSolder -> Capacitor_SMD:C_0402_1005Metric
- moved L1 0.44 mm to (119.9, 83.9)
- moved C5 0.30 mm to (122.1, 85.5)
- moved R5 0.26 mm to (119.9, 80.5)
- moved D1 0.20 mm to (102.3, 84.0)
- moved C4 0.10 mm to (121.1, 85.5)
Routing:
- net EN: track 43.4 -> 44.2 mm

Commit message: Add files via upload
Parts:
- C1, C2, C3, C4, C5, C6, C7, D1, R5, R6, R7: footprint Capacitor_SMD:C_0402_1005Metric -> Capacitor_SMD:C_0603_1608Metric
- moved R7 2.13 mm to (104.3, 85.3)
- moved C5 1.42 mm to (123.5, 85.5)
- moved C4 0.87 mm to (122.0, 85.5)
- moved C2 0.84 mm to (111.7, 86.3)
- moved C3 0.70 mm to (119.0, 85.5)
- moved L1 0.60 mm to (120.5, 83.9)
- moved C1 0.17 mm to (113.3, 86.1)
Routing:
- net +3.3V: track 22.1 -> 24.1 mm
- net +5V: track 68.8 -> 70.6 mm
- net Net-(D1-A): track 1.07 -> 2.09 mm
- net Net-(U2-FB): track 5.46 -> 6.13 mm
- net GND: track 42.0 -> 42.7 mm

Commit message: Add files via upload
Routing:
- net GND: track 42.7 -> 51.0 mm, vias 7 -> 9
- net I01: track 10.7 -> 11.5 mm
- net I02: track 9.15 -> 9.31 mm, vias 1 -> 0
- added copper zone on B.Cu, net (none)
- added copper zone on F.Cu, net (none)
Other:
- outline, holes or cut-outs redrawn
- board text added: "3.3V"
- board text added: "5V"
- board text added: "BOOT"
- board text added: "EN"
- board text added: "GND"
- board text added: "IO.01"
- board text added: "IO.02"
- board text added: "IO.03"
- board text added: "IO.04"
- board text added: "IO.05"
- board text added: "IO.06"
- board text added: "IO.07"
- board text added: "IO.08"
- board text added: "IO.09"
- board text added: "IO.10"
- board text added: "IO.11"
- board text added: "IO.12"
- board text added: "IO.13"
- board text added: "IO.14"
- board text added: "IO.15"
- board text added: "IO.16"
- board text added: "IO.17"
- board text added: "IO.18"
- board text added: "IO.21"
- board text added: "IO.35"
- board text added: "IO.36"
- board text added: "IO.37"
- board text added: "IO.38"
- board text added: "IO.39"
- board text added: "IO.40"
- board text added: "IO.41"
- board text added: "IO.42"
- board text added: "IO.45"
- board text added: "IO.46"
- board text added: "IO.47"
- board text added: "IO.48"
- board text added: "RX"
- board text added: "TX"
